Commit message: in launch_sim choice between controllers ,lidar noise,lastly made wheels collision be sphers and reduced friction,

File: description/lidar.xacro (robot description, xacro)
@@ -41,4 +41,9 @@
                     <max>12</max>
                 </range>
+                <noise>
+                    <type>gaussian</type> <!-- Gaussian noise, can also use 'uniform' -->
+                    <mean>0.0</mean> <!-- Mean value of the noise -->
+                    <stddev>0.02</stddev> <!-- Standard deviation (controls noise intensity) -->
+                </noise>
             </ray>
             <plugin name="laser_controller" filename="libgazebo_ros_ray_sensor.so">

File: description/robot.urdf.xacro (robot description, xacro)
@@ -1,7 +1,12 @@
 <?xml version="1.0"?>
 <robot xmlns:xacro="http://www.ros.org/wiki/xacro"  name="robot">
+    <xacro:arg name="use_ros2_control" default="true"/>
+    <xacro:if value="$(arg use_ros2_control)">
+    <xacro:include filename="ros2_control.xacro"/>
+    </xacro:if>
+    <xacro:unless value= "$(arg use_ros2_control)" >
+    <xacro:include filename="gazebo_control.xacro"/>
+    </xacro:unless>
     <xacro:include filename="robot_core.xacro"/>
-    <!-- <xacro:include filename="gazebo_control.xacro"/> -->
     <xacro:include filename="lidar.xacro"/>
-    <xacro:include filename="ros2_control.xacro"/>
 </robot>

File: description/robot_core.xacro (robot description, xacro)
@@ -2,4 +2,7 @@
 <robot xmlns:xacro="http://www.ros.org/wiki/xacro">
     <xacro:include filename="inertial_macros.xacro" />
+<!-- adding the variable -->
+    <xacro:property name="wheel_radius" value="0.05"/>
+    <xacro:property name="wheel_thick" value="0.04"/>
     <material name="white">
         <color rgba="1.0 1.0 1.0 1.0" />
@@ -36,4 +39,12 @@
                 <box size="0.6 0.3 0.2" />
             </geometry>
+                <surface>
+        <friction>
+            <ode>
+                <mu>1.00</mu>   <!-- Reduce friction -->
+                <mu2>0.25</mu2> <!-- Reduce friction -->
+            </ode>
+        </friction>
+    </surface>
         </collision>
         <xacro:inertial_box mass="0.5" x="0.6" y="0.3" z="0.2">
@@ -54,5 +65,5 @@
         <visual>
             <geometry>
-                <cylinder radius="0.05" length="0.04" />
+                <cylinder radius="${wheel_radius}" length="0.04" />
                 <material name="black" />
             </geometry>
@@ -60,8 +71,16 @@
         <collision>
             <geometry>
-                <cylinder radius="0.05" length="0.04" />
+                <sphere radius="${wheel_radius}"  />
             </geometry>
+                <surface>
+        <friction>
+            <ode>
+                <mu>1.00</mu>   <!-- Reduce friction -->
+                <mu2>0.25</mu2> <!-- Reduce friction -->
+            </ode>
+        </friction>
+    </surface>
         </collision>
-        <xacro:inertial_cylinder mass="0.1" length="0.04" radius="0.05">
+        <xacro:inertial_cylinder mass="0.1" length="0.04" radius="${wheel_radius}">
             <origin xyz="0.0 0.0 0.0" rpy="0.0 0.0 0.0" />
         </xacro:inertial_cylinder>
@@ -80,5 +99,5 @@
         <visual>
             <geometry>
-                <cylinder radius="0.05" length="0.04" />
+                <cylinder radius="${wheel_radius}" length="0.04" />
                 <material name="black" />
             </geometry>
@@ -86,8 +105,16 @@
         <collision>
             <geometry>
-                <cylinder radius="0.05" length="0.04" />
+                <sphere radius="${wheel_radius}"  />
             </geometry>
+                <surface>
+        <friction>
+            <ode>
+                <mu>1.00</mu>   <!-- Reduce friction -->
+                <mu2>0.25</mu2> <!-- Reduce friction -->
+            </ode>
+        </friction>
+    </surface>
         </collision>
-        <xacro:inertial_cylinder mass="0.1" length="0.04" radius="0.05">
+        <xacro:inertial_cylinder mass="0.1" length="0.04" radius="${wheel_radius}">
             <origin xyz="0.0 0.0 0.0" rpy="0.0 0.0 0.0" />
         </xacro:inertial_cylinder>
@@ -106,5 +133,5 @@
         <visual>
             <geometry>
-                <cylinder radius="0.05" length="0.04" />
+                <cylinder radius="${wheel_radius}" length="0.04" />
                 <material name="black" />
             </geometry>
@@ -112,8 +139,8 @@
         <collision>
             <geometry>
-                <cylinder radius="0.05" length="0.04" />
+                <sphere radius="${wheel_radius}"  />
             </geometry>
         </collision>
-        <xacro:inertial_cylinder mass="0.1" length="0.04" radius="0.05">
+        <xacro:inertial_cylinder mass="0.1" length="0.04" radius="${wheel_radius}">
             <origin xyz="0.0 0.0 0.0" rpy="0.0 0.0 0.0" />
         </xacro:inertial_cylinder>
@@ -132,5 +159,5 @@
         <visual>
             <geometry>
-                <cylinder radius="0.05" length="0.04" />
+                <cylinder radius="${wheel_radius}" length="0.04" />
                 <material name="black" />
             </geometry>
@@ -138,8 +165,16 @@
         <collision>
             <geometry>
-                <cylinder radius="0.05" length="0.04" />
+                <sphere radius="${wheel_radius}"  />
             </geometry>
+                <surface>
+        <friction>
+            <ode>
+                <mu>1.00</mu>   <!-- Reduce friction -->
+                <mu2>0.25</mu2> <!-- Reduce friction -->
+            </ode>
+        </friction>
+    </surface>
         </collision>
-        <xacro:inertial_cylinder mass="0.1" length="0.04" radius="0.05">
+        <xacro:inertial_cylinder mass="0.1" length="0.04" radius="${wheel_radius}">
             <origin xyz="0.0 0.0 0.0" rpy="0.0 0.0 0.0" />
         </xacro:inertial_cylinder>
