Commit message: created manual controler,gazebo intergration,launch file and world file

File: description/robot.urdf.xacro (robot description, xacro)
@@ -2,3 +2,4 @@
 <robot xmlns:xacro="http://www.ros.org/wiki/xacro"  name="robot">
     <xacro:include filename="robot_core.xacro"/>
+    <xacro:include filename="gazebo_control.xacro"/>
 </robot>

File: description/robot_core.xacro (robot description, xacro)
@@ -41,4 +41,7 @@
         </xacro:inertial_box>
     </link>
+               <gazebo reference = 'chassis'>
+                <material>Gazebo/SkyBlue </material>
+            </gazebo>
     <!-- left wheel link -->
     <joint name="left_back_wheel_joint" type="continuous">
@@ -64,4 +67,7 @@
         </xacro:inertial_cylinder>
     </link>
+             <gazebo reference = 'left_back_wheel'>
+                <material>Gazebo/Black</material>
+            </gazebo>
     <!-- right wheel link -->
     <joint name="right_back_wheel_joint" type="continuous">
@@ -87,4 +93,7 @@
         </xacro:inertial_cylinder>
     </link>
+                 <gazebo reference = 'right_back_wheel'>
+                <material>Gazebo/Black</material>
+            </gazebo>
     <!-- right front wheel link -->
     <joint name="right_front_wheel_joint" type="continuous">
@@ -110,4 +119,7 @@
         </xacro:inertial_cylinder>
     </link>
+                     <gazebo reference = 'right_front_wheel'>
+                <material>Gazebo/Black</material>
+            </gazebo>
     <!-- left wheel link -->
     <joint name="left_front_wheel_joint" type="continuous">
@@ -133,3 +145,6 @@
         </xacro:inertial_cylinder>
     </link>
+                         <gazebo reference = 'left_front_wheel'>
+                <material>Gazebo/Black</material>
+            </gazebo>
 </robot>

Commit message: added camera to simulation, added launch file for real robot, added ros2 control package parameters and calibrated the encoder counts per pid loops only# todo:calibrate the wheel radius and wheel separation

File: description/robot.urdf.xacro (robot description, xacro)
@@ -10,3 +10,4 @@
     <xacro:include filename="robot_core.xacro"/>
     <xacro:include filename="lidar.xacro"/>
+    <xacro:include filename="camera.xacro"/>
 </robot>

File: description/ros2_control.xacro (robot description, xacro)
@@ -1,9 +1,49 @@
 <?xml version="1.0"?>
 <robot xmlns:xacro="http://www.ros.org/wiki/xacro">
-    <ros2_control name="GazeboSystem" type="system">
-        <hardware>
-            <plugin>gazebo_ros2_control/GazeboSystem</plugin>
-        </hardware>
-        <joint name="left_back_wheel_joint">
+        <ros2_control name="RealRobot" type="system">
+            <hardware>
+                <plugin>diffdrive_arduino/DiffDriveArduino</plugin>
+                <param name="left_wheel_name">left_front_wheel_joint</param>
+                <param name="right_wheel_name">right_front_wheel_joint</param>
+                <param name="loop_rate">30</param>
+                <param name="device">/dev/ttyUSB1</param>
+                <param name="baud_rate">57600</param>
+                <param name="timeout">1000</param>
+                <param name="enc_counts_per_rev">1975</param>
+            </hardware>
+            <joint name="left_front_wheel_joint">
+                <command_interface name="velocity">
+                    <param name="min">-10</param>
+                    <param name="max"> 10</param>
+                </command_interface>
+                <state_interface name="velocity" />
+                <state_interface name="position" />
+            </joint>
+            <joint name="right_front_wheel_joint">
+                <command_interface name="velocity">
+                    <param name="min">-10</param>
+                    <param name="max"> 10</param>
+                </command_interface>
+                <state_interface name="velocity" />
+                <state_interface name="position" />
+            </joint>
+            <!-- <joint name="right_front_wheel_joint">
+                <command_interface name="velocity">
+                    <param name="min">-10</param>
+                    <param name="max"> 10</param>
+                </command_interface>
+                <state_interface name="velocity" />
+                <state_interface name="position" />
+            </joint>
+            <joint name="left_front_wheel_joint">
+                <command_interface name="velocity">
+                    <param name="min">-10</param>
+                    <param name="max"> 10</param>
+                </command_interface>
+                <state_interface name="velocity" />
+                <state_interface name="position" />
+            </joint> -->
+        </ros2_control>
+<!-- <joint name="left_back_wheel_joint">
             <command_interface name="velocity">
                 <param name="min">-10</param>
@@ -37,9 +77,10 @@
             <state_interface name="position" />
         </joint>
-    </ros2_control>
+    </ros2_control> -->
+<!--
     <gazebo>
         <plugin name="back_wheel" filename="libgazebo_ros2_control.so">
             <parameters>$(find akhmad_bot)/config/my_controllers.yaml</parameters>
         </plugin>
-    </gazebo>
+    </gazebo> -->
 </robot>
