Commit message: added mapping files and added the twist mux yaml

File: description/robot_core.xacro (robot description, xacro)
@@ -18,6 +18,12 @@
     </material>
     <!-- base link -->
-    <link name="base_link">
-    </link>
+    <link name="base_link"></link>
+    <!-- base_footprint link -->
+    <joint name="base_footprint_joint" type="fixed">
+        <parent link="base_link"/>
+        <child link="base_footprint"/>
+        <origin xyz="0.0 0.0 0.0" rpy="0.0 0.0 0.0"/>
+    </joint>
+    <link name="base_footprint"></link>
     <!-- chassis link -->
     <joint name="chassis_joint" type="fixed">

Commit message: calibrated the wheel separation and radius for acurate odometry, todo: update the urdf and get the mapping to work

File: description/robot_core.xacro (robot description, xacro)
@@ -30,9 +30,9 @@
         <parent link="base_link" />
         <child link="chassis" />
-        <origin xyz="-0.1 0.0 0.0" />
+        <origin xyz="0.1 0.0 0.0" />
     </joint>
     <link name="chassis">
         <visual>
-            <origin xyz="0.3 0.0 0.1" />
+            <origin xyz="-0.3 0.0 0.1" />
             <geometry>
                 <box size="0.6 0.3 0.2" />
@@ -65,5 +65,5 @@
         <parent link="base_link" />
         <child link="left_back_wheel" />
-        <origin xyz="0.0 0.175 0.0" rpy="-${pi/2} 0 0" />
+        <origin xyz="-0.4 0.175 0.0" rpy="-${pi/2} 0 0" />
         <axis xyz="0.0 0.0 1.0" />
     </joint>
@@ -99,5 +99,5 @@
         <parent link="base_link" />
         <child link="right_back_wheel" />
-        <origin xyz="0.0 -0.175 0.0" rpy="${pi/2} 0 0" />
+        <origin xyz="-0.4 -0.175 0.0" rpy="${pi/2} 0 0" />
         <axis xyz="0.0 0.0 -1.0" />
     </joint>
@@ -133,5 +133,5 @@
         <parent link="base_link" />
         <child link="right_front_wheel" />
-        <origin xyz="0.4 -0.175 0.0" rpy="${pi/2} 0 0" />
+        <origin xyz="0.0 -0.175 0.0" rpy="${pi/2} 0 0" />
         <axis xyz="0.0 0.0 -1.0" />
     </joint>
@@ -159,5 +159,5 @@
         <parent link="base_link" />
         <child link="left_front_wheel" />
-        <origin xyz="0.4 0.175 0.0" rpy="-${pi/2} 0 0" />
+        <origin xyz="0.0 0.175 0.0" rpy="-${pi/2} 0 0" />
         <axis xyz="0.0 0.0 1.0" />
     </joint>

File: description/ros2_control.xacro (robot description, xacro)
@@ -7,5 +7,5 @@
                 <param name="right_wheel_name">right_front_wheel_joint</param>
                 <param name="loop_rate">30</param>
-                <param name="device">/dev/ttyUSB1</param>
+                <param name="device">/dev/ttyUSB0</param>
                 <param name="baud_rate">57600</param>
                 <param name="timeout">1000</param>
